Commit message: Update my-robot.xacro

File: src/lab4_description/urdf/my-robot.xacro (robot description, xacro)
@@ -6,5 +6,5 @@
             <origin rpy="0 0 0" xyz="0.0 0.0 0.0" />
             <geometry>
-                <mesh filename="package://example_description/meshes/link_0.stl" />
+                <mesh filename="file:///$(find lab4_description)/meshes/link_0.stl" />
             </geometry>
         </visual>
@@ -14,5 +14,5 @@
             <origin rpy="0 0 0" xyz="0.0 0.0 0.0" />
             <geometry>
-                <mesh filename="package://example_description/meshes/link_1.stl" />
+                <mesh filename="file:///$(find lab4_description)/meshes/link_1.stl" />
             </geometry>
         </visual>
@@ -29,5 +29,5 @@
             <origin rpy="${pi} 0 0" xyz="0.0 0.0 0.0" />
             <geometry>
-                <mesh filename="package://example_description/meshes/link_2.stl" />
+                <mesh filename="file:///$(find lab4_description)/meshes/link_2.stl" />
             </geometry>
         </visual>
@@ -44,5 +44,5 @@
             <origin rpy="${pi} 0 0" xyz="0.0 0.0 0.0" />
             <geometry>
-                <mesh filename="package://example_description/meshes/link_3.stl" />
+                <mesh filename="file:///$(find lab4_description)/meshes/link_3.stl" />
             </geometry>
         </visual>
@@ -59,5 +59,5 @@
             <origin rpy="0 1.57 0" xyz="0.0 0.0 0.0" />
             <geometry>
-                <mesh filename="package://example_description/meshes/end_effector.stl" />
+                <mesh filename="file:///$(find lab4_description)/meshes/end_effector.stl" />
             </geometry>
         </visual>

Commit message: Update my-robot.xacro

File: src/lab4_description/urdf/my-robot.xacro (robot description, xacro)
@@ -6,5 +6,5 @@
             <origin rpy="0 0 0" xyz="0.0 0.0 0.0" />
             <geometry>
-                <mesh filename="file:///$(find lab4_description)/meshes/link_0.stl" />
+                <mesh filename="package://lab4_description/meshes/link_0.stl" />
             </geometry>
         </visual>
@@ -14,5 +14,5 @@
             <origin rpy="0 0 0" xyz="0.0 0.0 0.0" />
             <geometry>
-                <mesh filename="file:///$(find lab4_description)/meshes/link_1.stl" />
+                <mesh filename="package://lab4_description/meshes/link_1.stl" />
             </geometry>
         </visual>
@@ -29,5 +29,5 @@
             <origin rpy="${pi} 0 0" xyz="0.0 0.0 0.0" />
             <geometry>
-                <mesh filename="file:///$(find lab4_description)/meshes/link_2.stl" />
+                <mesh filename="package://lab4_description/meshes/link_2.stl" />
             </geometry>
         </visual>
@@ -44,5 +44,5 @@
             <origin rpy="${pi} 0 0" xyz="0.0 0.0 0.0" />
             <geometry>
-                <mesh filename="file:///$(find lab4_description)/meshes/link_3.stl" />
+                <mesh filename="package://lab4_description/meshes/link_3.stl" />
             </geometry>
         </visual>
@@ -59,5 +59,5 @@
             <origin rpy="0 1.57 0" xyz="0.0 0.0 0.0" />
             <geometry>
-                <mesh filename="file:///$(find lab4_description)/meshes/end_effector.stl" />
+                <mesh filename="package://lab4_description/meshes/end_effector.stl" />
             </geometry>
         </visual>
